Commit message: color coded walls in separate rooms

File: urdf/env.urdf (robot description, URDF)
Before this commit: robot env, 8 links, 7 joints
Links:
- removed link wall_1
- removed link wall_3
- removed link wall_4
- removed link wall_5
- added link wall_1_1, mass 1; collision box size=2.5 0.1 1.0; visual box size=2.5 0.1 1.0
- added link wall_1_2, mass 1; collision box size=2.5 0.1 1.0; visual box size=2.5 0.1 1.0
- added link wall_3_1, mass 1; collision box size=2.5 0.1 1.0; visual box size=2.5 0.1 1.0
- added link wall_3_2, mass 1; collision box size=2.5 0.1 1.0; visual box size=2.5 0.1 1.0
- added link wall_4_1, mass 1; collision box size=1.5 0.05 1.0; visual box size=1.5 0.05 1.0
- added link wall_4_2, mass 1; collision box size=1.5 0.05 1.0; visual box size=1.5 0.05 1.0
- added link wall_5_1, mass 1; collision box size=1.5 0.05 1.0; visual box size=1.5 0.05 1.0
- added link wall_5_2, mass 1; collision box size=1.5 0.05 1.0; visual box size=1.5 0.05 1.0
Joints:
- removed joint base_to_wall_1
- removed joint base_to_wall_3
- removed joint base_to_wall_4
- removed joint base_to_wall_5
- added joint base_to_wall_1_1: type fixed, parent base_link, child wall_1_1, origin xyz=2.55 0 0 rpy=0 0 1.571
- added joint base_to_wall_1_2: type fixed, parent base_link, child wall_1_2, origin xyz=2.55 0 0 rpy=0 0 1.571
- added joint base_to_wall_3_1: type fixed, parent base_link, child wall_3_1, origin xyz=-2.55 0 0 rpy=0 0 1.571
- added joint base_to_wall_3_2: type fixed, parent base_link, child wall_3_2, origin xyz=-2.55 0 0 rpy=0 0 1.571
- added joint base_to_wall_4_1: type fixed, parent base_link, child wall_4_1, origin xyz=1.75 0 0
- added joint base_to_wall_4_2: type fixed, parent base_link, child wall_4_2, origin xyz=1.75 0 0
- added joint base_to_wall_5_1: type fixed, parent base_link, child wall_5_1, origin xyz=-1.75 0 0
- added joint base_to_wall_5_2: type fixed, parent base_link, child wall_5_2, origin xyz=-1.75 0 0
