Commit message: added bin with hardcoded mesh path

File: urdf/trash_can.urdf (robot description, URDF)
Before this commit: robot trash_can, 1 links, 0 joints
Links:
- removed link base_link
- added link trash_can, mass 0.4193; collision mesh filename=/home/kchura01/catkin_ws/src/locobot_custom/urdf/meshes/tra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 scale=7 7 7; visual mesh filename=/home/kchura01/catkin_ws/src/locobot_custom/urdf/meshes/tra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 scale=7 7 7
